File: hardware/schematic/urine_analyzer_lite.kicad_sch (KiCad schematic)
At the start: 0 parts

Commit message: Stage 4: generate ERC-validated KiCad schematic from netlist model
- hardware/schematic/gen_schematic.py: rewritten to emit a real, connected schematic
  (replaces the old graphical mock-up generator); imports ../netlist model as source of truth
- urine_analyzer_lite.kicad_sch: machine-generated, connection-by-global-label
- Validated with KiCad 10 kicad-cli: ERC 0 errors; exported netlist matches model 39/39 nets
- Add rendered PDF + ERC_report.txt + README explaining validation and engineer next steps

Generic embedded symbols + placeholder footprints (the 59 ERC warnings) are for the engineer
to replace/assign. Electrically correct per the model; physical design needs engineer sign-off.

Co-Authored-By: Claude Opus 4.7 <noreply@anthropic.com>
Parts:
- added BT1: LiPo 3.7V 2000mAh, Connector:JST_PH_2pin, symbol ual:BT1
- added C1: 1000uF/10V, CP_Radial_D10.0mm_P5.00mm, symbol ual:C1
- added C2: 470uF/10V, CP_Radial_D8.0mm_P3.50mm, symbol ual:C2
- added C3: 10uF/10V, Capacitor_SMD:C_0805, symbol ual:C3
- added D1: High-CRI 95+ LED, LED_THT:LED_D5.0mm, symbol ual:D1
- added D2: 275nm UVC module, Module:UVC_LED_module, symbol ual:D2
- added LCD1: 3.5in SPI TFT ILI9488 +touch, Connector:TFT_SPI_14pin, symbol ual:LCD1
- added M1: GA12-N20 6V 200RPM +enc, Motor:GA12-N20_encoder, symbol ual:M1
- added PR1: CSN-A2 thermal, Connector:Printer_TTL_3pin, symbol ual:PR1
- added Q1: 2N7000, Package_TO_SOT_THT:TO-92, symbol ual:Q1
- added R1: 10k, Resistor_SMD:R_0805, symbol ual:R1
- added R2: 100R, Resistor_SMD:R_0805, symbol ual:R2
- added R3: 220R, Resistor_SMD:R_0805, symbol ual:R3
- added R4: 100k, Resistor_SMD:R_0805, symbol ual:R4
- added R5: 100k, Resistor_SMD:R_0805, symbol ual:R5
- added RT1: NTC 10k B3950, Resistor_THT:R_Axial_DIN0207, symbol ual:RT1
- added SW1: KW12-3, Button_Switch_THT:SW_Limit, symbol ual:SW1
- added SW2: KW12-3, Button_Switch_THT:SW_Limit, symbol ual:SW2
- added SW3: Tactile 6x6, Button_Switch_THT:SW_PUSH_6mm, symbol ual:SW3
- added U1: ESP32-S3-DevKitC-1, Module:ESP32-S3-DevKitC-1_header_2x22, symbol ual:U1
- added U10: HX711 1kg kit, Module:HX711_breakout, symbol ual:U10
- added U11: TCA9548A, Package_SO:TSSOP-24_4.4x7.8mm_P0.65mm, symbol ual:U11
- added U12: AMS1117-3.3, Package_TO_SOT_223:SOT-223-3_TabPin2, symbol ual:U12
- added U2: TP4056 USB-C, Module:TP4056_USBC, symbol ual:U2
- added U3: S13V25F5 buck-boost, Module:Pololu_S13V25Fx, symbol ual:U3
- added U4: TCS34725, Module:Adafruit_TCS34725, symbol ual:U4
- added U5: TCS34725, Module:Adafruit_TCS34725, symbol ual:U5
- added U6: SHT31-D, Module:SHT31_breakout, symbol ual:U6
- added U7: BH1750, Module:BH1750_breakout, symbol ual:U7
- added U8: ADS1115, Module:ADS1115_breakout, symbol ual:U8
- added U9: MX1508, Module:MX1508_driver, symbol ual:U9
Connections:
- net ENC_A: now also M1.C1, U1.6 (GPIO6)
- net ENC_B: now also M1.C2, U1.7 (GPIO7)
- net GND: now also BT1.2 (-), C1.2 (-), C2.2 (-), C3.2, D2.GND, LCD1.GND, M1.GND, PR1.GND, Q1.S, R1.2, R4.2, R5.2, SW1.1 (COM), SW2.1 (COM), SW3.2, U1.GND1 (GND), U1.GND2 (GND), U10.GND, U11.A0, U11.A1, U11.A2, U11.GND, U12.1 (GND), U2.2 (GND), U2.4 (BAT-), U2.6 (OUT-), U3.2 (GND), U4.GND, U5.GND, U6.ADR, U6.GND, U7.ADDR, U7.GND, U8.ADDR, U8.GND, U9.GND
- net I2C_SCL: now also U1.2 (GPIO2), U11.SCL, U6.SCL, U7.SCL, U8.SCL
- net I2C_SDA: now also U1.1 (GPIO1), U11.SDA, U6.SDA, U7.SDA, U8.SDA
- net LED_PWM: now also R3.1, U1.12 (GPIO12)
- net MOTOR_A: now also M1.M1, U9.OUT1
- net MOTOR_B: now also M1.M2, U9.OUT2
- net SCAN_BTN: now also SW3.1, U1.16 (GPIO16)
- net UVC_EN: now also D2.EN, R5.1, U1.13 (GPIO13)
- new net +3V3: C3.1, M1.VCC, RT1.1, U10.VCC, U11.RST (RESET), U11.VCC, U12.2 (VOUT), U4.VIN, U5.VIN, U6.VIN, U7.VCC, U8.VDD
- new net +5V: C1.1 (+), C2.1 (+), D1.A, D2.VIN, LCD1.VCC, PR1.VH, U1.5V, U12.3 (VIN), U3.3 (VOUT), U3.4 (EN), U9.VCC
- new net HX_DT: U1.14 (GPIO14), U10.DT
- new net HX_SCK: U1.15 (GPIO15), U10.SCK
- new net LED_DRAIN: Q1.D, R2.2
- new net LED_GATE: Q1.G, R3.2, R4.1
- new net LED_NODE: D1.K, R2.1
- new net LIM_END: SW2.2 (NO), U1.11 (GPIO11)
- new net LIM_HOME: SW1.2 (NO), U1.10 (GPIO10)
- new net MOT_IN1: U1.4 (GPIO4), U9.IN1
- new net MOT_IN2: U1.5 (GPIO5), U9.IN2
- new net NTC_SENSE: R1.1, RT1.2, U8.A0
- new net PRN_RX: PR1.TX, U1.18 (GPIO18)
- new net PRN_TX: PR1.RX, U1.17 (GPIO17)
- new net TCS1_SCL: U11.SC0, U4.SCL
- new net TCS1_SDA: U11.SD0, U4.SDA
- new net TCS2_SCL: U11.SC1, U5.SCL
- new net TCS2_SDA: U11.SD1, U5.SDA
- new net TFT_BL: LCD1.LED, U1.47 (GPIO47)
- new net TFT_CS: LCD1.CS, U1.41 (GPIO41)
- new net TFT_DC: LCD1.DC, U1.42 (GPIO42)
- new net TFT_MISO: LCD1.SDO, LCD1.T_DO, U1.40 (GPIO40)
- new net TFT_MOSI: LCD1.SDI, LCD1.T_DIN, U1.39 (GPIO39)
- new net TFT_RST: LCD1.RESET, U1.21 (GPIO21)
- new net TFT_SCLK: LCD1.SCK, LCD1.T_CLK, U1.38 (GPIO38)
- new net TOUCH_CS: LCD1.T_CS, U1.48 (GPIO48)
- new net VBAT: BT1.1 (+), U2.3 (BAT+)
- new net VBUS: U2.1 (VBUS)
- new net VSYS: U2.5 (OUT+), U3.1 (VIN)
Other:
- note removed: "275nm UVC LED"
- note removed: "2N7000 N-Ch MOSFET"
- note removed: "3.7V 2000mAh LiPo"
- note removed: "3V3"
- note removed: "5V"
- note removed: "A"
- note removed: "A+"
- note removed: "A-"
- note removed: "ADDR"
- note removed: "ADS1115 ADC"
- note removed: "AIN0"
- note removed: "ALRT"
- note removed: "B+"
- note removed: "B-"
- note removed: "BH1750 Light Sensor"
- note removed: "BT1"
- note removed: "COM"
- note removed: "CSN-A2 Thermal Printer"
- note removed: "D"
- note removed: "D0+"
- note removed: "D0-"
- note removed: "D1"
- note removed: "D2"
- note removed: "DCLK"
- note removed: "DT"
- note removed: "E+"
- note removed: "E-"
- note removed: "EN"
- note removed: "ENC_A"
- note removed: "ENC_B"
- note removed: "ESP32-S3-DevKitC-1"
- note removed: "FS1"
- note removed: "G"
- note removed: "GND"
- note removed: "GPIO1"
- note removed: "GPIO10"
- note removed: "GPIO11"
- note removed: "GPIO12"
- note removed: "GPIO13"
- note removed: "GPIO14"
- note removed: "GPIO15"
- note removed: "GPIO16"
- note removed: "GPIO17"
- note removed: "GPIO18"
- note removed: "GPIO19"
- note removed: "GPIO2"
- note removed: "GPIO21"
- note removed: "GPIO22"
- note removed: "GPIO3"
- note removed: "GPIO4"
- note removed: "GPIO5"
- note removed: "GPIO6"
- note removed: "GPIO7"
- note removed: "GPIO8"
- note removed: "GPIO9"
- note removed: "HX711 Load Cell Amp"
- note removed: "High-CRI LED 95+ CRI"
- note removed: "IN1"
- note removed: "IN2"
- note removed: "INT"
- note removed: "K"
- note removed: "KW12-3 End Limit"
- note removed: "KW12-3 Home Limit"
- note removed: "LCD1"
- note removed: "LED"
- note removed: "Load Cell 1kg"
- note removed: "M+"
- note removed: "M-"
- note removed: "M1"
- note removed: "MX1508 H-Bridge"
- note removed: "N20 DC Motor+Encoder"
- note removed: "NO"
- note removed: "NTC Thermistor 10k"
- note removed: "OUT+"
- note removed: "OUT-"
- note removed: "OUT1"
- note removed: "OUT2"
- note removed: "P1"
- note removed: "P2"
- note removed: "PR1"
- note removed: "Q1"
- note removed: "RT1"
- note removed: "RX"
- note removed: "S"
- note removed: "S13V25F5 5V Reg"
- note removed: "SCK"
- note removed: "SCL"
- note removed: "SDA"
- note removed: "SHT31-D Env Sensor"
- note removed: "SW1"
- note removed: "SW2"
- note removed: "SW3"
- note removed: "Scan Button 6x6mm"
- note removed: "T1"
- note removed: "T2"
- note removed: "TCS34725 RGB #1"
- note removed: "TCS34725 RGB #2"
- note removed: "TP4056 USB-C Charger"
- note removed: "TX"
- note removed: "U1"
- note removed: "U10"
- note removed: "U2"
- note removed: "U3"
- note removed: "U4"
- note removed: "U5"
- note removed: "U6"
- note removed: "U7"
- note removed: "U8"
- note removed: "U9"
- note removed: "USB_IN+"
- note removed: "USB_IN-"
- note removed: "VCC"
- note removed: "VDD"
- note removed: "VH"
- note removed: "VIN"
- note removed: "VOUT"
- note removed: "Waveshare 4.3in DSI LCD"
- company: Levram Lifesciences -> (none)
- title: Urine Analyzer Lite — Schematic -> (none)

Commit message: Stage 4: real symbols + footprints, and a starting PCB
- hardware/footprints.py: real KiCad footprints for all 31 parts (modules = 2.54mm pin
  headers, pin order to verify vs datasheets; LED/TO-92 pad overrides)
- schematic: 14 jellybean discretes now use real Device:/Switch: library symbols (embedded);
  modules/MOSFET stay custom but numbered by PCB pad; every part carries a real footprint.
  ERC 0 errors; netlist matches model 39/39 by ref+pad
- hardware/pcb/: starting board built via pcbnew Python (build_pcb.py) — 31 footprints
  placed + net-assigned + outline; schematic-parity 0; unrouted ratsnest + cosmetic auto-grid
  DRC only. Includes project, 3D render, DRC report
- netlist generator now emits real footprints + pad numbers

Validated with KiCad 10.0.3. Starting board for engineer verification — confirm module pin
order, place/route, power planes, DRC->0, Gerbers.

Co-Authored-By: Claude Opus 4.7 <noreply@anthropic.com>
Parts:
- removed BT1: LiPo 3.7V 2000mAh, Connector:JST_PH_2pin, symbol ual:BT1
- removed C1: 1000uF/10V, CP_Radial_D10.0mm_P5.00mm, symbol ual:C1
- removed C2: 470uF/10V, CP_Radial_D8.0mm_P3.50mm, symbol ual:C2
- removed C3: 10uF/10V, Capacitor_SMD:C_0805, symbol ual:C3
- removed D1: High-CRI 95+ LED, LED_THT:LED_D5.0mm, symbol ual:D1
- removed R1: 10k, Resistor_SMD:R_0805, symbol ual:R1
- removed R2: 100R, Resistor_SMD:R_0805, symbol ual:R2
- removed R3: 220R, Resistor_SMD:R_0805, symbol ual:R3
- removed R4: 100k, Resistor_SMD:R_0805, symbol ual:R4
- removed R5: 100k, Resistor_SMD:R_0805, symbol ual:R5
- removed RT1: NTC 10k B3950, Resistor_THT:R_Axial_DIN0207, symbol ual:RT1
- removed SW1: KW12-3, Button_Switch_THT:SW_Limit, symbol ual:SW1
- removed SW2: KW12-3, Button_Switch_THT:SW_Limit, symbol ual:SW2
- removed SW3: Tactile 6x6, Button_Switch_THT:SW_PUSH_6mm, symbol ual:SW3
- added BT1: LiPo 3.7V 2000mAh, Connector_JST:JST_PH_S2B-PH-K_1x02_P2.00mm_Horizontal, symbol Device:Battery_Cell
- added C1: 1000uF/10V, Capacitor_THT:CP_Radial_D10.0mm_P5.00mm, symbol Device:C_Polarized
- added C2: 470uF/10V, Capacitor_THT:CP_Radial_D8.0mm_P3.50mm, symbol Device:C_Polarized
- added C3: 10uF/10V, Capacitor_SMD:C_0805_2012Metric, symbol Device:C
- added D1: High-CRI 95+ LED, LED_THT:LED_D5.0mm_Clear, symbol Device:LED
- added R1: 10k, Resistor_SMD:R_0805_2012Metric, symbol Device:R
- added R2: 100R, Resistor_SMD:R_0805_2012Metric, symbol Device:R
- added R3: 220R, Resistor_SMD:R_0805_2012Metric, symbol Device:R
- added R4, R5: 100k, Resistor_SMD:R_0805_2012Metric, symbol Device:R
- added RT1: NTC 10k B3950, Resistor_THT:R_Axial_DIN0207_L6.3mm_D2.5mm_P7.62mm_Horizontal, symbol Device:Thermistor
- added SW1, SW2: KW12-3, Connector_PinHeader_2.54mm:PinHeader_1x02_P2.54mm_Vertical, symbol Switch:SW_Push
- added SW3: Tactile 6x6, Connector_PinHeader_2.54mm:PinHeader_1x02_P2.54mm_Vertical, symbol Switch:SW_Push
- D2: footprint Module:UVC_LED_module -> Connector_PinHeader_2.54mm:PinHeader_1x03_P2.54mm_Vertical
- LCD1: footprint Connector:TFT_SPI_14pin -> Connector_PinHeader_2.54mm:PinHeader_1x13_P2.54mm_Vertical
- M1: footprint Motor:GA12-N20_encoder -> Connector_PinHeader_2.54mm:PinHeader_1x06_P2.54mm_Vertical
- PR1: footprint Connector:Printer_TTL_3pin -> Connector_PinHeader_2.54mm:PinHeader_1x04_P2.54mm_Vertical
- Q1: footprint Package_TO_SOT_THT:TO-92 -> Package_TO_SOT_THT:TO-92_Inline
- U1: footprint Module:ESP32-S3-DevKitC-1_header_2x22 -> Connector_PinHeader_2.54mm:PinHeader_2x22_P2.54mm_Vertical
- U10: footprint Module:HX711_breakout -> Connector_PinHeader_2.54mm:PinHeader_1x04_P2.54mm_Vertical
- U11: footprint Package_SO:TSSOP-24_4.4x7.8mm_P0.65mm -> Connector_PinHeader_2.54mm:PinHeader_1x12_P2.54mm_Vertical
- U12: footprint Package_TO_SOT_223:SOT-223-3_TabPin2 -> Package_TO_SOT_SMD:SOT-223-3_TabPin2
- U2: footprint Module:TP4056_USBC -> Connector_PinHeader_2.54mm:PinHeader_1x06_P2.54mm_Vertical
- U3: footprint Module:Pololu_S13V25Fx -> Connector_PinHeader_2.54mm:PinHeader_1x04_P2.54mm_Vertical
- U4, U5: footprint Module:Adafruit_TCS34725 -> Connector_PinHeader_2.54mm:PinHeader_1x04_P2.54mm_Vertical
- U6: footprint Module:SHT31_breakout -> Connector_PinHeader_2.54mm:PinHeader_1x05_P2.54mm_Vertical
- U7: footprint Module:BH1750_breakout -> Connector_PinHeader_2.54mm:PinHeader_1x05_P2.54mm_Vertical
- U8: footprint Module:ADS1115_breakout -> Connector_PinHeader_2.54mm:PinHeader_1x06_P2.54mm_Vertical
- U9: footprint Module:MX1508_driver -> Connector_PinHeader_2.54mm:PinHeader_1x06_P2.54mm_Vertical
Connections:
- net +3V3: now also M1.3 (VCC), U10.1 (VCC), U11.1 (VCC), U11.5 (RESET), U4.1 (VIN), U5.1 (VIN), U6.1 (VIN), U7.1 (VCC), U8.1 (VDD), C3.1, RT1.1; no longer M1.VCC, U10.VCC, U11.RST (RESET), U11.VCC, U4.VIN, U5.VIN, U6.VIN, U7.VCC, U8.VDD
- net +5V: now also D2.1 (VIN), LCD1.1 (VCC), PR1.1 (VH), U1.1 (5V), U9.1 (VCC), C1.1, C2.1, D1.2 (A); no longer D2.VIN, LCD1.VCC, PR1.VH, U1.5V, U9.VCC
- net ENC_A: now also M1.5 (C1), U1.8 (GPIO6); no longer M1.C1, U1.6 (GPIO6)
- net ENC_B: now also M1.6 (C2), U1.9 (GPIO7); no longer M1.C2, U1.7 (GPIO7)
- net GND: now also D2.2 (GND), LCD1.2 (GND), M1.4 (GND), PR1.2 (GND), Q1.1 (S), U1.2 (GND), U1.3 (GND), U10.2 (GND), U11.2 (GND), U11.6 (A0), U11.7 (A1), U11.8 (A2), U4.2 (GND), U5.2 (GND), U6.2 (GND), U6.5 (ADR), U7.2 (GND), U7.5 (ADDR), U8.2 (GND), U8.5 (ADDR), U9.2 (GND), BT1.2 (-), C1.2, C2.2, C3.2, R1.2, R4.2, R5.2, SW1.1, SW2.1, SW3.2; no longer D2.GND, LCD1.GND, M1.GND, PR1.GND, Q1.S, U1.GND1 (GND), U1.GND2 (GND), U10.GND, U11.A0, U11.A1, U11.A2, U11.GND, U4.GND, U5.GND, U6.ADR, U6.GND, U7.ADDR, U7.GND, U8.ADDR, U8.GND, U9.GND
- net HX_DT: now also U10.3 (DT); no longer U10.DT
- net HX_SCK: now also U10.4 (SCK); no longer U10.SCK
- net I2C_SCL: now also U1.5 (GPIO2), U11.4 (SCL), U6.4 (SCL), U7.4 (SCL), U8.4 (SCL); no longer U1.2 (GPIO2), U11.SCL, U6.SCL, U7.SCL, U8.SCL
- net I2C_SDA: now also U1.4 (GPIO1), U11.3 (SDA), U6.3 (SDA), U7.3 (SDA), U8.3 (SDA); no longer U1.1 (GPIO1), U11.SDA, U6.SDA, U7.SDA, U8.SDA
- net LED_DRAIN: now also Q1.3 (D), R2.2; no longer Q1.D
- net LED_GATE: now also Q1.2 (G), R3.2, R4.1; no longer Q1.G
- net LED_NODE: now also D1.1 (K), R2.1
- net LED_PWM: now also R3.1
- net LIM_END: now also SW2.2
- net LIM_HOME: now also SW1.2
- net MOTOR_A: now also M1.1 (M1), U9.5 (OUT1); no longer M1.M1, U9.OUT1
- net MOTOR_B: now also M1.2 (M2), U9.6 (OUT2); no longer M1.M2, U9.OUT2
- net MOT_IN1: now also U1.6 (GPIO4), U9.3 (IN1); no longer U1.4 (GPIO4), U9.IN1
- net MOT_IN2: now also U1.7 (GPIO5), U9.4 (IN2); no longer U1.5 (GPIO5), U9.IN2
- net NTC_SENSE: now also U8.6 (A0), R1.1, RT1.2; no longer U8.A0
- net PRN_RX: now also PR1.4 (TX); no longer PR1.TX
- net PRN_TX: now also PR1.3 (RX); no longer PR1.RX
- net SCAN_BTN: now also SW3.1
- net TCS1_SCL: now also U11.10 (SC0), U4.4 (SCL); no longer U11.SC0, U4.SCL
- net TCS1_SDA: now also U11.9 (SD0), U4.3 (SDA); no longer U11.SD0, U4.SDA
- net TCS2_SCL: now also U11.12 (SC1), U5.4 (SCL); no longer U11.SC1, U5.SCL
- net TCS2_SDA: now also U11.11 (SD1), U5.3 (SDA); no longer U11.SD1, U5.SDA
- net TFT_BL: now also LCD1.8 (LED), U1.25 (GPIO47); no longer LCD1.LED, U1.47 (GPIO47)
- net TFT_CS: now also LCD1.3 (CS), U1.23 (GPIO41); no longer LCD1.CS, U1.41 (GPIO41)
- net TFT_DC: now also LCD1.5 (DC), U1.24 (GPIO42); no longer LCD1.DC, U1.42 (GPIO42)
- net TFT_MISO: now also LCD1.13 (T_DO), LCD1.9 (SDO), U1.22 (GPIO40); no longer LCD1.SDO, LCD1.T_DO, U1.40 (GPIO40)
- net TFT_MOSI: now also LCD1.12 (T_DIN), LCD1.6 (SDI), U1.21 (GPIO39); no longer LCD1.SDI, LCD1.T_DIN, U1.39 (GPIO39)
- net TFT_RST: now also LCD1.4 (RESET), U1.19 (GPIO21); no longer LCD1.RESET, U1.21 (GPIO21)
- net TFT_SCLK: now also LCD1.10 (T_CLK), LCD1.7 (SCK), U1.20 (GPIO38); no longer LCD1.SCK, LCD1.T_CLK, U1.38 (GPIO38)
- net TOUCH_CS: now also LCD1.11 (T_CS), U1.26 (GPIO48); no longer LCD1.T_CS, U1.48 (GPIO48)
- net UVC_EN: now also D2.3 (EN), R5.1; no longer D2.EN
- net VBAT: now also BT1.1 (+)
